Commit message: fix: change a0509 frame - world -> manipulator_base_link

File: dsr_description2/xacro/a0509.urdf.xacro (robot description, xacro)
@@ -15,9 +15,9 @@
   </xacro:if>
   <xacro:a0509 namespace="$(arg namespace)"/>
-  <link name="world" />
+  <link name="manipulator_base_link" />
   <!-- World fixed joint-->
   <joint name="world_fixed" type="fixed">
     <origin xyz="0 0 0" rpy="0 0 0"/>
-    <parent link="world"/>
+    <parent link="manipulator_base_link"/>
     <child link="base_link"/>
   </joint>

Commit message: fix: world frame deleted

File: dsr_description2/xacro/a0509.urdf.xacro (robot description, xacro)
@@ -15,11 +15,4 @@
   </xacro:if>
   <xacro:a0509 namespace="$(arg namespace)"/>
-  <link name="manipulator_base_link" />
-  <!-- World fixed joint-->
-  <joint name="world_fixed" type="fixed">
-    <origin xyz="0 0 0" rpy="0 0 0"/>
-    <parent link="manipulator_base_link"/>
-    <child link="base_link"/>
-  </joint>
   <xacro:if value="${gz}">
     <xacro:include filename="$(find dsr_description2)/ros2_control/a0509.gz_ros2_control.xacro" />
